File: 38-04-usb-sleuth.kicad_sch (KiCad schematic)
At the start: 64 parts, among them J1 Conn_1x05, J2 USB_C_12401832E402A, J3 USB_C_12401832E402A, J4 USB_Micro-B_KH-MICRO5P-JN, J5 USB_Mini-B_U-M-M5DD-W-1, J6 USB3_A_HC-USB3.0-L168-WP, SW1 SW_DPDT_x2, SW2 ZX-1.27BM-4PSMD, U1 STM32C031K6T6

Commit message: touch main.c
Connections:
- net A_GND_SENS renamed A_GND_SENSE
- net A_VBUS_SENS renamed A_VBUS_SENSE
- net B_CC1_SENS renamed B_CC1_SENSE
- net B_CC2_SENS renamed B_CC2_SENSE
Changed lines of the file:
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@@
     (effects (font (size 1.27 1.27)) (justify left bottom))
   )
-  (label "A_GND_SENS" (at 55.88 180.975 180) (fields_autoplaced)
+  (label "A_GND_SENSE" (at 55.88 180.975 180) (fields_autoplaced)
     (effects (font (size 1.27 1.27)) (justify right bottom))
   )
@@
     (effects (font (size 1.27 1.27)) (justify left bottom))
   )
-  (label "A_VBUS_SENS" (at 172.085 34.925 0) (fields_autoplaced)
+  (label "A_VBUS_SENSE" (at 172.085 34.925 0) (fields_autoplaced)
     (effects (font (size 1.27 1.27)) (justify left bottom))
   )
@@
     (effects (font (size 1.27 1.27)) (justify right bottom))
   )
-  (label "A_VBUS_SENS" (at 95.885 180.975 180) (fields_autoplaced)
+  (label "A_VBUS_SENSE" (at 95.885 180.975 180) (fields_autoplaced)
     (effects (font (size 1.27 1.27)) (justify right bottom))
   )
@@
     (effects (font (size 1.27 1.27)) (justify right bottom))
   )
-  (label "B_CC2_SENS" (at 196.85 147.32 180) (fields_autoplaced)
+  (label "B_CC2_SENSE" (at 196.85 147.32 180) (fields_autoplaced)
     (effects (font (size 1.27 1.27)) (justify right bottom))
   )
@@
     (effects (font (size 1.27 1.27)) (justify right bottom))
   )
-  (label "B_CC2_SENS" (at 184.785 45.085 180) (fields_autoplaced)
+  (label "B_CC2_SENSE" (at 184.785 45.085 180) (fields_autoplaced)
     (effects (font (size 1.27 1.27)) (justify right bottom))
   )
@@
     (effects (font (size 1.27 1.27)) (justify right bottom))
   )
-  (label "B_CC1_SENS" (at 135.255 139.7 0) (fields_autoplaced)
+  (label "B_CC1_SENSE" (at 135.255 139.7 0) (fields_autoplaced)
     (effects (font (size 1.27 1.27)) (justify left bottom))
   )
@@
     (effects (font (size 1.27 1.27)) (justify left bottom))
   )
-  (label "B_CC1_SENS" (at 184.785 42.545 180) (fields_autoplaced)
+  (label "B_CC1_SENSE" (at 184.785 42.545 180) (fields_autoplaced)
     (effects (font (size 1.27 1.27)) (justify right bottom))
   )
@@
     (effects (font (size 1.27 1.27)) (justify left bottom))
   )
-  (label "A_GND_SENS" (at 184.785 32.385 180) (fields_autoplaced)
-    (effects (font (size 1.27 1.27)) (justify right bottom))
-  )
+  (label "A_GND_SENSE" (at 184.785 32.385 180) (fields_autoplaced)
+    (effects (font (size 1.27 1.27)) (justify right bottom))
+  )

Commit message: update readme
Connections:
- net A_GND_SENSE renamed GND_SENSE
- net A_VBUS_SENSE renamed VBUS_SENSE
Other:
- note added: "Open for DMM Test"
- note removed: "Open SW2 A-D to test A and B side VBUS to GND, or Rp, Rd, Ra"
- moved on the sheet: C4, J1
