File: 38-04-usb-sleuth.kicad_pcb (KiCad board)
At the start: 2 copper layers, 90 x 90 mm, 68 parts, among them J1 Conn_1x05, J2 USB_C_12401832E402A, J3 USB_C_12401832E402A, J4 USB_Micro-B_KH-MICRO5P-JN, J5 USB_Mini-B_U-M-M5DD-W-1, J6 USB3_A_HC-USB3.0-L168-WP, SW1 SW_DPDT_x2, SW2 ZX-1.27BM-4PSMD, U1 STM32C031K6T6

Commit message: adding stm32ide project files and HAL Drivers
Other:
- board text added: "3.2"
- board text removed: "3.1"
Changed lines of the file:
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@@
     (effects (font (size 0.8 0.8) (thickness 0.15)))
   )
-  (gr_text "3.1" (at 143.7132 93.9038) (layer "F.SilkS")
+  (gr_text "3.2" (at 143.7132 93.9038) (layer "F.SilkS")
     (effects (font (size 1 1) (thickness 0.15)))
   )
